File: rp2040_stamp.kicad_sch (KiCad schematic)
At the start: 38 parts, among them J1 Conn_South, J2 Conn_North, J3 Conn_East, J4 Conn_West, Q1 BSS84, SW1 SW_RESET, U1 RP2040, U2 AP2112K-3.3, U3 W25Q64JV, U4 MCP73831, Y1 XYDBPCNANF-12MHZ

Commit message: simplify stamp
Parts:
- removed C16, C6, C7: 10uF, Capacitor_SMD:C_0603_1608Metric, symbol Device:C_Small
- removed D1: D_Schottky_Small, Diode_SMD:D_SOD-323, symbol Device:D_Schottky_Small
- removed D2: LED_CHR, LED_SMD:LED_0603_1608Metric, symbol Device:LED_Small
- removed D3: WS2812B-2020, LED_SMD_Extra:WS2812B-2020, symbol LED_Extra:WS2812B-2020
- removed JP1: Jumper_Neopixel_VDD, Jumper:SolderJumper-2_P1.3mm_Bridged_RoundedPad1.0x1.5mm, symbol Jumper:Jumper_2_Bridged
- removed JP2: Jumper_Neopixel, Jumper:SolderJumper-2_P1.3mm_Bridged_RoundedPad1.0x1.5mm, symbol Jumper:Jumper_2_Bridged
- removed Q1: BSS84, Package_TO_SOT_SMD:SOT-23, symbol Transistor_FET:BSS84
- removed R6: 100K, Resistor_SMD:R_0603_1608Metric, symbol Device:R_Small
- removed R7: 2K, Resistor_SMD:R_0603_1608Metric, symbol Device:R_Small
- removed R8: 1K, Resistor_SMD:R_0603_1608Metric, symbol Device:R_Small
- removed U2: AP2112K-3.3, Package_TO_SOT_SMD:SOT-23-5, symbol Regulator_Linear:AP2112K-3.3
- removed U4: MCP73831, Package_TO_SOT_SMD:SOT-23-5, symbol Battery_Management_Extra:MCP73831
- removed Y1: XYDBPCNANF-12MHZ, Crystal:Crystal_SMD_2520-4Pin_2.5x2.0mm, symbol Device:Crystal_GND24_Small
- added R4: 1k, Resistor_SMD:R_0603_1608Metric, symbol Device:R
- added Y1: Crystal, UserLib:Crystal_SMD_7040-2Pin_7.0x4.0mm, symbol Device:Crystal
- C1: renamed from C14; value 12pF -> 27pF
- C2: renamed from C15; value 12pF -> 27pF
- SW1: footprint Button_Switch_SMD:SW_SPST_B3U-1000P -> Jumper:SolderJumper-2_P1.3mm_Open_RoundedPad1.0x1.5mm
- U2: renamed from U1; footprint Package_DFN_QFN_Extra:QFN-56_EP_7x7_Pitch0.4mm -> UserLib:RP2040
- renumbered C12 to C10, C13 to C11, C1 to C3, C3 to C4, C4 to C5, C5 to C6, C8 to C7, C10 to C8, C11 to C9, J4 to J1, J1 to J3, J3 to J4, R5 to R1, R3 to R2, R4 to R3, R2 to R5, R1 to R6, U3 to U1
Connections:
- net at C1.1, U2.20 (XIN): now also Y1.1
- net at C2.1: now also R4.1, Y1.2; no longer U2.21 (XOUT)
- net ~QSPI_CS~ renamed ~{QSPI_CS}
- net ~RESET~ renamed ~{RESET}
- new net: R4.2, U2.21 (XOUT)
- no-connect marks 1 -> 0
Other:
- moved on the sheet: C1, C2, R1, U1
